Commit message: Add files via upload

File: left_arm_description/urdf/romo_left_arm.urdf (robot description, URDF)
Before this commit: robot romo_left_arm, 6 links, 5 joints
Links:
- added link grip_link, mass 0.2; collision mesh filename=package://romo_ros/meshes/left_chain_gripper_move.stl; visual mesh filename=package://romo_ros/meshes/left_chain_gripper_move.stl
- added link link6, mass 0.4; collision mesh filename=package://romo_ros/meshes/left_chain_link6.stl; visual mesh filename=package://romo_ros/meshes/left_chain_link6.stl
- added link link7, mass 0.4; collision mesh filename=package://romo_ros/meshes/left_chain_gripper_fix.stl; visual mesh filename=package://romo_ros/meshes/left_chain_gripper_fix.stl
Joints:
- added joint grip_joint: type revolute, parent link7, child grip_link, origin xyz=0.06 0.0 -0.015 rpy=0 0 0, axis 0 1 0, limit lower=-2.8274333886 upper=2.8274333886 effort=1000 velocity=6.5
- added joint joint5: type revolute, parent link5, child link6, origin xyz=0.036 0.0 0.0 rpy=0 0 0, axis 1 0 0, limit lower=-2.8274333886 upper=2.8274333886 effort=1000 velocity=6.5
- added joint joint6: type revolute, parent link6, child link7, origin xyz=0.22 0.0 0.0 rpy=0 0 0, axis 0 1 0, limit lower=-2.8274333886 upper=2.8274333886 effort=1000 velocity=6.5

File: left_arm_description/urdf/romo_left_arm.xacro (robot description, xacro)
@@ -208,37 +208,127 @@
     </inertial>
   </link>
+  <!--  Joint 5 -->
+  <joint name="joint5" type="revolute">
+    <parent link="link5"/>
+    <child link="link6"/>
+    <origin xyz="0.036 0.0 0.0" rpy="0 0 0"/>
+    <axis xyz="1 0 0"/>
+    <limit velocity="6.5" effort="1000" lower="${-pi*0.9}" upper="${pi*0.9}" />
+  </joint>
+  <!-- Transmission 5 -->
+  <transmission name="tran5">
+    <type>transmission_interface/SimpleTransmission</type>
+    <joint name="joint5">
+      <hardwareInterface>PositionJointInterface</hardwareInterface>
+    </joint>
+    <actuator name="motor5">
+      <hardwareInterface>PositionJointInterface</hardwareInterface>
+      <mechanicalReduction>1</mechanicalReduction>
+    </actuator>
+  </transmission>
+  <!--  Link 6 -->
+  <link name="link6">
+    <collision>
+      <origin xyz="-0.036 0.205 0.053" rpy="0 0 0"/>
+      <geometry>
+        <mesh filename="package://romo_ros/meshes/left_chain_link6.stl" />
+      </geometry>
+    </collision>
+    <visual>
+      <origin xyz="-0.036 0.205 0.053" rpy="0 0 0"/>
+      <geometry>
+        <mesh filename="package://romo_ros/meshes/left_chain_link6.stl" />
+      </geometry>
+      <material name="grey"/>
+    </visual>
+    <inertial>
+      <origin xyz="-0.036 0.205 0.053" />
+      <mass value="0.4" />
+      <inertia ixx="0.001" ixy="0.0" ixz="0.0"
+               iyy="0.001" iyz="0.0"
+               izz="0.001" />
+    </inertial>
+  </link>
+  <!--  Joint 6 -->
+  <joint name="joint6" type="revolute">
+    <parent link="link6"/>
+    <child link="link7"/>
+    <origin xyz="0.22 0.0 0.0" rpy="0 0 0"/>
+    <axis xyz="0 1 0"/>
+    <limit velocity="6.5" effort="1000" lower="${-pi*0.9}" upper="${pi*0.9}" />
+  </joint>
+  <!-- Transmission 6 -->
+  <transmission name="tran6">
+    <type>transmission_interface/SimpleTransmission</type>
+    <joint name="joint6">
+      <hardwareInterface>PositionJointInterface</hardwareInterface>
+    </joint>
+    <actuator name="motor6">
+      <hardwareInterface>PositionJointInterface</hardwareInterface>
+      <mechanicalReduction>1</mechanicalReduction>
+    </actuator>
+  </transmission>
+  <!--  Link 7 -->
+  <link name="link7">
+    <collision>
+      <origin xyz="-0.256 0.205 0.053" rpy="0 0 0"/>
+      <geometry>
+        <mesh filename="package://romo_ros/meshes/left_chain_gripper_fix.stl" />
+      </geometry>
+    </collision>
+    <visual>
+      <origin xyz="-0.256 0.205 0.053" rpy="0 0 0"/>
+      <geometry>
+        <mesh filename="package://romo_ros/meshes/left_chain_gripper_fix.stl" />
+      </geometry>
+      <material name="grey"/>
+    </visual>
+    <inertial>
+      <origin xyz="-0.256 0.205 0.053" />
+      <mass value="0.4" />
+      <inertia ixx="0.001" ixy="0.0" ixz="0.0"
+               iyy="0.001" iyz="0.0"
+               izz="0.001" />
+    </inertial>
+  </link>
+  <!--  grip_joint -->
+  <joint name="grip_joint" type="revolute">
+    <parent link="link7"/>
+    <child link="grip_link"/>
+    <origin xyz="0.06 0.0 -0.015" rpy="0 0 0"/>
+    <axis xyz="0 1 0"/>
+    <limit velocity="6.5" effort="1000" lower="${-pi*0.9}" upper="${pi*0.9}" />
+  </joint>
   <!--  Grip link -->
-  <!--<link name="grip_link">
-    <collision>
-      <origin xyz="0.0 0.047 0" rpy="0 0 0"/>
-      <geometry>
-        <mesh filename="package://romo_ros/meshes/left_chain_link_grip_l.stl" scale="0.001 0.001 0.001"/>
-      </geometry>
-    </collision>
-    <visual>
-      <origin xyz="0.0 0.047 0" rpy="0 0 0"/>
-      <geometry>
-        <mesh filename="package://romo_ros/meshes/left_chain_link_grip_l.stl" scale="0.001 0.001 0.001"/>
-      </geometry>
-      <material name="grey"/>
-    </visual>
-    <inertial>
-      <origin xyz="0 0 0" />
-      <mass value="0.01" />
-      <inertia ixx="0.001" ixy="0.0" ixz="0.0"
-               iyy="0.001" iyz="0.0"
-               izz="0.001" />
-    </inertial>
-  </link>
-  -->
+  <link name="grip_link">
+    <collision>
+      <origin xyz="-0.316 0.205 0.068" rpy="0 0 0"/>
+      <geometry>
+        <mesh filename="package://romo_ros/meshes/left_chain_gripper_move.stl" />
+      </geometry>
+    </collision>
+    <visual>
+      <origin xyz="-0.316 0.205 0.068" rpy="0 0 0"/>
+      <geometry>
+        <mesh filename="package://romo_ros/meshes/left_chain_gripper_move.stl" />
+      </geometry>
+      <material name="grey"/>
+    </visual>
+    <inertial>
+      <origin xyz="-0.316 0.205 0.068" />
+      <mass value="0.2" />
+      <inertia ixx="0.001" ixy="0.0" ixz="0.0"
+               iyy="0.001" iyz="0.0"
+               izz="0.001" />
+    </inertial>
+  </link>
   <!--  Grip joint -->
-  <!--<joint name="grip_joint" type="prismatic">
-    <parent link="link5"/>
+  <!--<joint name="grip_joint" type="revolute">
+    <parent link="link7"/>
     <child link="grip_link"/>
-    <origin xyz="0.071 0.0 0.0" rpy="0 0 0"/>
-    <axis xyz="0 -1 0"/>
-    <limit velocity="6.5" effort="1000" lower="-0.01" upper="0.035" />
-  </joint>
-  -->
+    <origin xyz="0.0 0.0 0.0" rpy="0 0 0"/>
+    <axis xyz="1 0 0"/>
+    <limit velocity="6.5" effort="1000" lower="${-pi*0.9}" upper="${pi*0.9}" />
+  </joint>-->
   <!-- Transmission 5 -->
   <!--<transmission name="tran5">
